File: LM3886x2_inv_bal_servo.kicad_pcb (KiCad board)
At the start: 2 copper layers, 125 x 60 mm, 69 parts, among them J1 INPUT, J2 OUT, J3 36V, J4 15V, U1 NE5532, U2 NE5532, U3 OPA2134, U4 LM3886, U5 LM3886

Commit message: finished PCB layout
Parts:
- added H1: MountingHole, MountingHole:MountingHole_3.2mm_M3_Pad_Via, F.Cu at (61.2, 106.2)
- added H2: MountingHole, MountingHole:MountingHole_3.2mm_M3_Pad_Via, F.Cu at (178.8, 106.2)
- added H3: MountingHole, MountingHole:MountingHole_3.2mm_M3_Pad_Via, F.Cu at (61.2, 56.2)
- added H4: MountingHole, MountingHole:MountingHole_3.2mm_M3_Pad_Via, F.Cu at (178.8, 56.2)
- R5: value 1M -> 2M2
- moved R8 3.00 mm to (163.0, 82.5)
- moved R3 2.50 mm to (172.5, 82.5)
- moved R28 0.75 mm to (97.5, 71.8)
Routing:
- net +15V: track 177.2 -> 170.7 mm
- net Net-(R3-Pad1): track 12.0 -> 6.52 mm
- net GND: track 45.7 -> 48.2 mm, vias 23 -> 453
- net +36V: track 0.00 -> 2.26 mm, vias 0 -> 36
- net Net-(R8-Pad1): track 15.7 -> 13.4 mm
- net Net-(R10-Pad2): track 14.0 -> 12.1 mm
- net /U1SIG+: track 26.2 -> 27.8 mm
- net /U1SIG-: track 24.2 -> 25.1 mm
- net -15V: track 91.0 -> 90.1 mm, vias 4 -> 8
- net Net-(C19-Pad1): track 28.9 -> 29.6 mm
- net /U5OUT: track 22.0 -> 21.4 mm
- net -36V: vias 0 -> 24
- added copper zone on B.Cu, net +36V
- added copper zone on F.Cu, net +36V
- added copper zone on B.Cu, net -36V
- added copper zone on F.Cu, net GND
Other:
- board text added: "+15V"
- board text added: "+36V"
- board text added: "-15V"
- board text added: "-36V"
- board text added: "GND"
- board text added: "IN+"
- board text added: "IN-"
- board text added: "July 2023"
- board text added: "LM3886/2876 in parallel, inverted input, servo offset adjust"
- board text added: "OUT+"
- board text added: "Pavlo’s Lab"
- board text added: "Rev1.0"
